File: Wahly_KiCAD/Microcontroller.sch (KiCad schematic (older format))
At the start: 18 parts, among them U5 STM32F302C8Tx, Y1 16MHz

Commit message: updates
Parts:
- added D4: Red, LED_SMD:LED_0603_1608Metric, symbol Device:LED_Small
- added R9: 10k, Resistor_SMD:R_0603_1608Metric, symbol Device:R_Small
- added SW1: SW_SPDT, Button_Switch_SMD:SW_SPDT_PCM12, symbol Switch:SW_SPDT
- D2: renamed from D?; footprint (none) -> LED_SMD:LED_0603_1608Metric
- R5: renamed from R?; footprint (none) -> Resistor_SMD:R_0402_1005Metric
- gave numbers to parts that had none: 1
Connections:
- net +3V3: now also SW1.1 (A)
- net BOOT0: now also R9.2
- net GND: now also D4.1 (K), SW1.3 (C)
- net I2C1_SCL: now also U5.42 (PB6); no longer U5.38 (PA15)
- net TEMP_INT: now also U5.45 (PB8); no longer U5.42 (PB6)
- net ADC1_IN1: now reaches U5.10 (PA0)
- net ADC1_IN2: now reaches U5.11 (PA1)
- net TIM2_CH3: now reaches U5.12 (PA2)
- net TIM2_CH4: now reaches U5.13 (PA3)
- net at U5.18 (PB0): no longer D2.2 (A)
- net at U5.30 (PA9): now also D2.2 (A)
- net SWD_SWO: now reaches U5.39 (PB3)
- new net: D4.2 (A), R9.1, SW1.2 (B)
- no-connect marks 0 -> 13
Other:
- moved on the sheet: D2, R5
Changed lines of the file:
@@
 Text GLabel 1700 4900 0    50   Input ~ 0
 I2C1_SDA
-Text GLabel 3700 5700 2    50   Input ~ 0
+Text GLabel 1700 4800 0    50   Input ~ 0
 I2C1_SCL
 Wire Wire Line
-	3700 5700 3400 5700
-Wire Wire Line
 	2100 4900 1700 4900
-$Comp
-L Device:R_Small R1
-U 1 1 6182CDED
-P 9200 3650
-F 0 "R1" H 9259 3696 50  0000 L CNN
-F 1 "2k2" H 9259 3605 50  0000 L CNN
-F 2 "Resistor_SMD:R_0603_1608Metric" H 9200 3650 50  0001 C CNN
-F 3 "~" H 9200 3650 50  0001 C CNN
-	1    9200 3650
-	1    0    0    -1
-$EndComp
 $Comp
 L Device:R_Small R2
@@
 Text Notes 8550 1000 0    79   ~ 16
 High Speed External Crystal
-Text GLabel 1700 4800 0    50   Input ~ 0
+Text GLabel 1700 5000 0    50   Input ~ 0
 TEMP_INT
 Wire Wire Line
@@
 STM32F3 Microcontroller
 $Comp
-L Device:LED_Small D?
+L Device:LED_Small D2
 U 1 1 618E1479
-P 900 4400
-F 0 "D?" V 946 4330 50  0000 R CNN
-F 1 "Red" V 855 4330 50  0000 R CNN
-F 2 "" V 900 4400 50  0001 C CNN
-F 3 "~" V 900 4400 50  0001 C CNN
-	1    900  4400
+P 4450 5350
+F 0 "D2" V 4496 5280 50  0000 R CNN
+F 1 "Red" V 4405 5280 50  0000 R CNN
+F 2 "LED_SMD:LED_0603_1608Metric" V 4450 5350 50  0001 C CNN
+F 3 "~" V 4450 5350 50  0001 C CNN
+	1    4450 5350
 	0    -1   -1   0
 $EndComp
 $Comp
-L Device:R_Small R?
+L Device:R_Small R5
 U 1 1 618E2C5F
-P 900 4650
-F 0 "R?" H 959 4696 50  0000 L CNN
-F 1 "1k" H 959 4605 50  0000 L CNN
-F 2 "" H 900 4650 50  0001 C CNN
-F 3 "~" H 900 4650 50  0001 C CNN
-	1    900  4650
-	1    0    0    -1
-$EndComp
-$Comp
-L power:GND #PWR?
+P 4450 5600
+F 0 "R5" H 4509 5646 50  0000 L CNN
+F 1 "1k" H 4509 5555 50  0000 L CNN
+F 2 "Resistor_SMD:R_0402_1005Metric" H 4450 5600 50  0001 C CNN
+F 3 "~" H 4450 5600 50  0001 C CNN
+	1    4450 5600
+	1    0    0    -1
+$EndComp
+$Comp
+L power:GND #PWR0130
 U 1 1 618E3325
-P 900 4800
-F 0 "#PWR?" H 900 4550 50  0001 C CNN
-F 1 "GND" H 905 4627 50  0000 C CNN
-F 2 "" H 900 4800 50  0001 C CNN
-F 3 "" H 900 4800 50  0001 C CNN
-	1    900  4800
-	1    0    0    -1
-$EndComp
-Wire Wire Line
-	900  4800 900  4750
-Wire Wire Line
-	900  4550 900  4500
-Wire Wire Line
-	900  4200 2100 4200
-Wire Wire Line
-	900  4200 900  4300
-$Comp
-L Memory_Flash:W25Q32JVSS U?
+P 4450 5750
+F 0 "#PWR0130" H 4450 5500 50  0001 C CNN
+F 1 "GND" H 4455 5577 50  0000 C CNN
+F 2 "" H 4450 5750 50  0001 C CNN
+F 3 "" H 4450 5750 50  0001 C CNN
+	1    4450 5750
+	1    0    0    -1
+$EndComp
+Wire Wire Line
+	4450 5750 4450 5700
+Wire Wire Line
+	4450 5500 4450 5450
+$Comp
+L Memory_Flash:W25Q32JVSS U6
 U 1 1 618ED2B7
 P 9000 5350
-F 0 "U?" H 8650 5950 50  0000 C CNN
+F 0 "U6" H 8650 5950 50  0000 C CNN
 F 1 "W25Q32JVSS" H 8600 5850 50  0000 C CNN
 F 2 "Package_SO:SOIC-8_5.23x5.23mm_P1.27mm" H 9000 5350 50  0001 C CNN
@@
 	9750 5150 9500 5150
 $Comp
-L power:GND #PWR?
+L power:GND #PWR0131
 U 1 1 61901CF6
 P 9000 5800
-F 0 "#PWR?" H 9000 5550 50  0001 C CNN
+F 0 "#PWR0131" H 9000 5550 50  0001 C CNN
 F 1 "GND" H 9005 5627 50  0000 C CNN
 F 2 "" H 9000 5800 50  0001 C CNN
@@
 $EndComp
 $Comp
-L power:+3.3V #PWR?
+L power:+3.3V #PWR0132
 U 1 1 619020AD
 P 9000 4900
-F 0 "#PWR?" H 9000 4750 50  0001 C CNN
+F 0 "#PWR0132" H 9000 4750 50  0001 C CNN
 F 1 "+3.3V" H 9015 5073 50  0000 C CNN
 F 2 "" H 9000 4900 50  0001 C CNN
@@
 Wire Wire Line
 	9500 5550 9750 5550
+$Comp
+L Switch:SW_SPDT SW1
+U 1 1 617F404A
+P 6900 3300
+F 0 "SW1" H 6900 3585 50  0000 C CNN
+F 1 "SW_SPDT" H 6900 3494 50  0000 C CNN
+F 2 "Button_Switch_SMD:SW_SPDT_PCM12" H 6900 3300 50  0001 C CNN
+F 3 "~" H 6900 3300 50  0001 C CNN
+	1    6900 3300
+	1    0    0    -1
+$EndComp
+$Comp
+L power:+3.3V #PWR0133
+U 1 1 617F4944
+P 7200 3050
+F 0 "#PWR0133" H 7200 2900 50  0001 C CNN
+F 1 "+3.3V" H 7215 3223 50  0000 C CNN
+F 2 "" H 7200 3050 50  0001 C CNN
+F 3 "" H 7200 3050 50  0001 C CNN
+	1    7200 3050
+	1    0    0    -1
+$EndComp
+$Comp
+L power:GND #PWR0134
+U 1 1 617F4F38
+P 7200 3650
+F 0 "#PWR0134" H 7200 3400 50  0001 C CNN
+F 1 "GND" H 7205 3477 50  0000 C CNN
+F 2 "" H 7200 3650 50  0001 C CNN
+F 3 "" H 7200 3650 50  0001 C CNN
+	1    7200 3650
+	1    0    0    -1
+$EndComp
+Wire Wire Line
+	7200 3650 7200 3400
+Wire Wire Line
+	7200 3400 7100 3400
+Wire Wire Line
+	7100 3200 7200 3200
+Wire Wire Line
+	7200 3200 7200 3050
+$Comp
+L Device:R_Small R1
+U 1 1 6182CDED
+P 9200 3650
+F 0 "R1" H 9259 3696 50  0000 L CNN
+F 1 "2k2" H 9259 3605 50  0000 L CNN
+F 2 "Resistor_SMD:R_0603_1608Metric" H 9200 3650 50  0001 C CNN
+F 3 "~" H 9200 3650 50  0001 C CNN
+	1    9200 3650
+	1    0    0    -1
+$EndComp
+$Comp
+L Device:R_Small R9
+U 1 1 61803704
+P 6400 3300
+F 0 "R9" V 6204 3300 50  0000 C CNN
+F 1 "10k" V 6295 3300 50  0000 C CNN
+F 2 "Resistor_SMD:R_0603_1608Metric" H 6400 3300 50  0001 C CNN
+F 3 "~" H 6400 3300 50  0001 C CNN
+	1    6400 3300
+	0    1    1    0
+$EndComp
+Wire Wire Line
+	6700 3300 6600 3300
+Text GLabel 6200 3300 0    50   Input ~ 0
+BOOT0
+Wire Wire Line
+	6300 3300 6200 3300
+$Comp
+L power:GND #PWR0135
+U 1 1 6180AC3C
+P 6600 3650
+F 0 "#PWR0135" H 6600 3400 50  0001 C CNN
+F 1 "GND" H 6605 3477 50  0000 C CNN
+F 2 "" H 6600 3650 50  0001 C CNN
+F 3 "" H 6600 3650 50  0001 C CNN
+	1    6600 3650
+	1    0    0    -1
+$EndComp
+$Comp
+L Device:LED_Small D4
+U 1 1 6181584A
+P 6600 3500
+F 0 "D4" V 6646 3430 50  0000 R CNN
+F 1 "Red" V 6555 3430 50  0000 R CNN
+F 2 "LED_SMD:LED_0603_1608Metric" V 6600 3500 50  0001 C CNN
+F 3 "~" V 6600 3500 50  0001 C CNN
+	1    6600 3500
+	0    -1   -1   0
+$EndComp
+Wire Wire Line
+	6600 3650 6600 3600
+Wire Wire Line
+	6600 3400 6600 3300
+Connection ~ 6600 3300
+Wire Wire Line
+	6600 3300 6500 3300
+Wire Wire Line
+	1700 5000 2100 5000
+Wire Wire Line
+	3400 5100 4450 5100
+Wire Wire Line
+	4450 5100 4450 5250
+Wire Notes Line
+	5650 2650 5650 4000
+Wire Notes Line
+	5650 4000 7600 4000
+Wire Notes Line
+	7600 4000 7600 2650
+Wire Notes Line
+	7600 2650 5650 2650
+Wire Notes Line
+	7450 4550 7450 6150
+Wire Notes Line
+	7450 6150 10400 6150
+Wire Notes Line
+	10400 6150 10400 4550
+Wire Notes Line
+	7450 4550 10400 4550
+Text GLabel 1700 4500 0    50   Input ~ 0
+SWD_SWO
+Wire Wire Line
+	2100 4500 1700 4500
+Text GLabel 3700 4200 2    50   Input ~ 0
+ADC1_IN1
+Text GLabel 3700 4300 2    50   Input ~ 0
+ADC1_IN2
+Wire Wire Line
+	3400 4200 3700 4200
+Wire Wire Line
+	3700 4300 3400 4300
+Text GLabel 3700 4400 2    50   Input ~ 0
+TIM2_CH3
+Text GLabel 3700 4500 2    50   Input ~ 0
+TIM2_CH4
+Wire Wire Line
+	3700 4500 3400 4500
+Wire Wire Line
+	3400 4400 3700 4400
+NoConn ~ 2100 3800
+NoConn ~ 2100 3900
+NoConn ~ 2100 4000
+NoConn ~ 2100 4200
+NoConn ~ 2100 4600
+NoConn ~ 2100 4700
+NoConn ~ 2100 5100
+NoConn ~ 2100 5200
+NoConn ~ 2100 5300
+NoConn ~ 3400 5700
+NoConn ~ 3400 5200
+NoConn ~ 3400 5000
+NoConn ~ 3400 4600
 $EndSCHEMATC

Commit message: pdf schematic
Parts:
- R3: footprint Resistor_SMD:R_0603_1608Metric -> Resistor_SMD:R_0402_1005Metric
Other:
- note added: "BOOT0"
- note added: "FLASH"
- moved on the sheet: C13, C14, D4, R1, R2, R3, R9, SW1, U6, Y1
