File: Wahly_KiCAD/Power.sch (KiCad schematic (older format))
At the start: 7 parts, among them J1 USB_B_Micro, U1 LM1117-3.3, U2 USBLC6-2SC6

Commit message: updates
Parts:
- D1: renamed from D?; footprint (none) -> LED_SMD:LED_0603_1608Metric
- R4: renamed from R?; footprint (none) -> Resistor_SMD:R_0402_1005Metric
Changed lines of the file:
@@
 3.3V LDO
 $Comp
-L Device:LED_Small D?
+L Device:LED_Small D1
 U 1 1 618DD8FE
 P 6850 4500
-F 0 "D?" V 6896 4430 50  0000 R CNN
+F 0 "D1" V 6896 4430 50  0000 R CNN
 F 1 "Green" V 6805 4430 50  0000 R CNN
-F 2 "" V 6850 4500 50  0001 C CNN
+F 2 "LED_SMD:LED_0603_1608Metric" V 6850 4500 50  0001 C CNN
 F 3 "~" V 6850 4500 50  0001 C CNN
 	1    6850 4500
@@
 $EndComp
 $Comp
-L power:+3.3V #PWR?
+L power:+3.3V #PWR0128
 U 1 1 618DE8AE
 P 6850 4300
-F 0 "#PWR?" H 6850 4150 50  0001 C CNN
+F 0 "#PWR0128" H 6850 4150 50  0001 C CNN
 F 1 "+3.3V" H 6865 4473 50  0000 C CNN
 F 2 "" H 6850 4300 50  0001 C CNN
@@
 $EndComp
 $Comp
-L Device:R_Small R?
+L Device:R_Small R4
 U 1 1 618DFAC8
 P 6850 4750
-F 0 "R?" H 6909 4796 50  0000 L CNN
+F 0 "R4" H 6909 4796 50  0000 L CNN
 F 1 "1k" H 6909 4705 50  0000 L CNN
-F 2 "" H 6850 4750 50  0001 C CNN
+F 2 "Resistor_SMD:R_0402_1005Metric" H 6850 4750 50  0001 C CNN
 F 3 "~" H 6850 4750 50  0001 C CNN
 	1    6850 4750
@@
 $EndComp
 $Comp
-L power:GND #PWR?
+L power:GND #PWR0129
 U 1 1 618DFDF5
 P 6850 4900
-F 0 "#PWR?" H 6850 4650 50  0001 C CNN
+F 0 "#PWR0129" H 6850 4650 50  0001 C CNN
 F 1 "GND" H 6855 4727 50  0000 C CNN
 F 2 "" H 6850 4900 50  0001 C CNN
