File: Wahly_KiCAD/Wahly.sch (KiCad schematic (older format))
At the start: 0 parts

Commit message: updates
Parts:
- added H1, H2, H3, H4: MountingHole_Pad, MountingHole:MountingHole_4.3mm_M4_Pad_Via, symbol Mechanical:MountingHole_Pad
Connections:
- new net GND: H1.1, H2.1, H3.1, H4.1
Changed lines of the file:
@@
 Text Notes 800  5600 0    98   ~ 20
 Connectors
+$Comp
+L Mechanical:MountingHole_Pad H1
+U 1 1 617ED9E8
+P 3700 2850
+F 0 "H1" H 3800 2899 50  0000 L CNN
+F 1 "MountingHole_Pad" H 3800 2808 50  0000 L CNN
+F 2 "MountingHole:MountingHole_4.3mm_M4_Pad_Via" H 3700 2850 50  0001 C CNN
+F 3 "~" H 3700 2850 50  0001 C CNN
+	1    3700 2850
+	1    0    0    -1
+$EndComp
+$Comp
+L Mechanical:MountingHole_Pad H2
+U 1 1 617EE5D0
+P 3700 3300
+F 0 "H2" H 3800 3349 50  0000 L CNN
+F 1 "MountingHole_Pad" H 3800 3258 50  0000 L CNN
+F 2 "MountingHole:MountingHole_4.3mm_M4_Pad_Via" H 3700 3300 50  0001 C CNN
+F 3 "~" H 3700 3300 50  0001 C CNN
+	1    3700 3300
+	1    0    0    -1
+$EndComp
+$Comp
+L Mechanical:MountingHole_Pad H3
+U 1 1 617EE80B
+P 3700 3750
+F 0 "H3" H 3800 3799 50  0000 L CNN
+F 1 "MountingHole_Pad" H 3800 3708 50  0000 L CNN
+F 2 "MountingHole:MountingHole_4.3mm_M4_Pad_Via" H 3700 3750 50  0001 C CNN
+F 3 "~" H 3700 3750 50  0001 C CNN
+	1    3700 3750
+	1    0    0    -1
+$EndComp
+$Comp
+L Mechanical:MountingHole_Pad H4
+U 1 1 617EEA48
+P 3700 4150
+F 0 "H4" H 3800 4199 50  0000 L CNN
+F 1 "MountingHole_Pad" H 3800 4108 50  0000 L CNN
+F 2 "MountingHole:MountingHole_4.3mm_M4_Pad_Via" H 3700 4150 50  0001 C CNN
+F 3 "~" H 3700 4150 50  0001 C CNN
+	1    3700 4150
+	1    0    0    -1
+$EndComp
+Wire Wire Line
+	3700 2950 3350 2950
+Wire Wire Line
+	3350 2950 3350 3400
+Wire Wire Line
+	3350 4250 3700 4250
+Wire Wire Line
+	3700 3850 3350 3850
+Connection ~ 3350 3850
+Wire Wire Line
+	3350 3850 3350 4250
+Wire Wire Line
+	3700 3400 3350 3400
+Connection ~ 3350 3400
+Wire Wire Line
+	3350 3400 3350 3850
+$Comp
+L power:GND #PWR0127
+U 1 1 617EF2A9
+P 3350 4350
+F 0 "#PWR0127" H 3350 4100 50  0001 C CNN
+F 1 "GND" H 3355 4177 50  0000 C CNN
+F 2 "" H 3350 4350 50  0001 C CNN
+F 3 "" H 3350 4350 50  0001 C CNN
+	1    3350 4350
+	1    0    0    -1
+$EndComp
+Wire Wire Line
+	3350 4350 3350 4250
+Connection ~ 3350 4250
 $EndSCHEMATC

Commit message: pdf schematic
Other:
- note added: "Mounting Holes"
Changed lines of the file:
@@
 encoding utf-8
 Sheet 1 5
-Title ""
+Title "Wahly Sensor Board - STM32"
 Date ""
-Rev ""
+Rev "0.1"
 Comp ""
 Comment1 ""
@@
 	3350 4350 3350 4250
 Connection ~ 3350 4250
+Wire Notes Line
+	2850 2500 2850 4700
+Wire Notes Line
+	2850 4700 4800 4700
+Wire Notes Line
+	4800 4700 4800 2500
+Wire Notes Line
+	4800 2500 2850 2500
+Text Notes 3450 2600 0    50   ~ 10
+Mounting Holes
 $EndSCHEMATC
