File: Wahly_KiCAD/Wahly.kicad_pcb (KiCad board)
At the start: 2 copper layers, 1 part, among them U1 STM32WB30CEU5A

Commit message: updates
Parts:
- added C1: 10uF, Capacitor_SMD:C_0402_1005Metric, F.Cu at (175.2, 107.4)
- added C10: 100nF, Capacitor_SMD:C_0402_1005Metric, F.Cu at (158.5, 106.5)
- added C11: 10nF, Capacitor_SMD:C_0402_1005Metric, F.Cu at (161.4, 108.4)
- added C12: 1uF, Capacitor_SMD:C_0402_1005Metric, F.Cu at (163.0, 99.8)
- added C13: 20pF, Capacitor_SMD:C_0402_1005Metric, F.Cu at (158.5, 110.4)
- added C14: 20pF, Capacitor_SMD:C_0402_1005Metric, F.Cu at (161.4, 106.5)
- added C15: 100nF, Capacitor_SMD:C_0402_1005Metric, F.Cu at (180.0, 84.1)
- added C2: 10uF, Capacitor_SMD:C_0402_1005Metric, F.Cu at (190.0, 97.2)
- added C3: 100nF, Capacitor_SMD:C_0402_1005Metric, F.Cu at (196.3, 93.7)
- added C4: 100nF, Capacitor_SMD:C_0402_1005Metric, F.Cu at (201.8, 93.2)
- added C5: 10uF, Capacitor_SMD:C_0402_1005Metric, F.Cu at (204.7, 93.2)
- added C6: 4,7uF, Capacitor_SMD:C_0402_1005Metric, F.Cu at (158.5, 108.4)
- added C7: 100nF, Capacitor_SMD:C_0402_1005Metric, F.Cu at (154.7, 110.9)
- added C8: 100nF, Capacitor_SMD:C_0402_1005Metric, F.Cu at (162.5, 103.7)
- added C9: 100nF, Capacitor_SMD:C_0402_1005Metric, F.Cu at (163.0, 101.8)
- added D1: Green, LED_SMD:LED_0603_1608Metric, F.Cu at (180.8, 104.7)
- added D2: Red, LED_SMD:LED_0603_1608Metric, F.Cu at (143.2, 108.9)
- added D4: Red, LED_SMD:LED_0603_1608Metric, F.Cu at (159.6, 97.5)
- added FB1: 600 @ 600MHz, Inductor_SMD:L_0603_1608Metric, F.Cu at (151.2, 111.1)
- added H1: MountingHole_Pad, MountingHole:MountingHole_4.3mm_M4_Pad_Via, F.Cu at (151.1, 86.1)
- added H2: MountingHole_Pad, MountingHole:MountingHole_4.3mm_M4_Pad_Via, F.Cu at (151.1, 76.0)
- added H3: MountingHole_Pad, MountingHole:MountingHole_4.3mm_M4_Pad_Via, F.Cu at (141.0, 86.1)
- added H4: MountingHole_Pad, MountingHole:MountingHole_4.3mm_M4_Pad_Via, F.Cu at (141.0, 76.0)
- added J1: USB_B_Micro, Connector_USB:USB_Micro-B_Molex-105017-0001, F.Cu at (183.7, 99.2)
- added J2: Power, Connector_PinHeader_2.54mm:PinHeader_1x04_P2.54mm_Vertical, F.Cu at (180.9, 73.2)
- added J3: ADC, Connector_PinHeader_2.54mm:PinHeader_1x04_P2.54mm_Vertical, F.Cu at (185.5, 73.2)
- added J4: SWD, Connector_PinHeader_1.27mm:PinHeader_2x05_P1.27mm_Vertical_SMD, F.Cu at (197.3, 75.1)
- added J5: TIM2, Connector_PinHeader_2.54mm:PinHeader_1x04_P2.54mm_Vertical, F.Cu at (190.2, 73.2)
- added R1: 2k2, Resistor_SMD:R_0603_1608Metric, F.Cu at (159.1, 104.2)
- added R10: 22, Resistor_SMD:R_0603_1608Metric, F.Cu at (194.5, 83.1)
- added R2: 2k2, Resistor_SMD:R_0603_1608Metric, F.Cu at (159.6, 100.1)
- added R3: 47, Resistor_SMD:R_0603_1608Metric, F.Cu at (143.2, 111.4)
- added R4: 1k, Resistor_SMD:R_0402_1005Metric, F.Cu at (175.2, 105.5)
- added R5: 1k, Resistor_SMD:R_0402_1005Metric, F.Cu at (163.1, 97.2)
- added R6: 22, Resistor_SMD:R_0603_1608Metric, F.Cu at (198.5, 83.1)
- added R7: 22, Resistor_SMD:R_0603_1608Metric, F.Cu at (198.5, 80.6)
- added R8: 22, Resistor_SMD:R_0603_1608Metric, F.Cu at (194.5, 80.6)
- added R9: 10k, Resistor_SMD:R_0603_1608Metric, F.Cu at (147.2, 111.1)
- added SW1: SW_SPDT, Button_Switch_SMD:SW_SPDT_PCM12, F.Cu at (152.2, 106.0)
- added U2: USBLC6-2SC6, Package_TO_SOT_SMD:SOT-23-6, F.Cu at (171.3, 106.8)
- added U3: SHT30-DIS, Sensor_Humidity:Sensirion_DFN-8-1EP_2.5x2.5mm_P0.5mm_EP1.1x1.7mm, F.Cu at (202.6, 90.2)
- added U4: LIS3DHTR, Package_LGA:LGA-16_3x3mm_P0.5mm, F.Cu at (192.9, 88.5)
- added U5: STM32F302C8Tx, Package_QFP:LQFP-48_7x7mm_P0.5mm, F.Cu at (141.6, 101.9)
- added U6: W25Q32JVSS, Package_SO:SOIC-8_5.23x5.23mm_P1.27mm, F.Cu at (152.4, 99.6)
- added Y1: 16MHz, Crystal:Crystal_SMD_TXC_7M-4Pin_3.2x2.5mm, F.Cu at (138.5, 109.8)
- U1: value STM32WB30CEU5A -> LM1117-3.3; footprint QFN50P700X700X60-49N -> Package_TO_SOT_SMD:SOT-223
- moved U1 27.9 mm to (173.8, 100.3)
Connections:
- U1 pad 1: Net-(U1-Pad1) -> GND
- U1 pad 2: Net-(U1-Pad2) -> +3V3
- U1 pad 3: Net-(U1-Pad3) -> +5V
- U1 pad 4: Net-(U1-Pad4) -> (no net)

Commit message: pdf schematic
Parts:
- R3: footprint Resistor_SMD:R_0603_1608Metric -> Resistor_SMD:R_0402_1005Metric
- moved R7 143.7 mm to (55.8, 96.9)
- moved R6 143.1 mm to (55.8, 94.3)
- moved J4 142.0 mm to (55.5, 80.5)
- moved U3 138.0 mm to (66.5, 67.3)
- moved J3 134.7 mm to (52.1, 91.8)
- moved J5 131.9 mm to (59.6, 91.8)
- moved R8 131.7 mm to (63.5, 94.3)
- moved R10 131.7 mm to (63.5, 96.8)
- moved C3 131.3 mm to (67.2, 69.7), turned to 180 degrees
- moved C5 123.8 mm to (80.9, 95.1), turned to 90 degrees
- moved C4 119.9 mm to (81.9, 95.1), turned to 90 degrees
- moved C2 111.0 mm to (79.0, 100.3), turned to 90 degrees
- moved J1 109.2 mm to (75.1, 111.2)
- moved J2 109.2 mm to (71.8, 66.5), turned to 90 degrees
- moved U4 108.7 mm to (84.3, 93.9), turned to 180 degrees
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Other:
- board outline added: 50.1 x 50.1 mm

Commit message: Silkscreen & DRC
Parts:
- moved J2 45.1 mm to (72.3, 111.5), turned to 270 degrees
- moved SW1 29.6 mm to (68.5, 67.9), turned to 180 degrees
- moved J4 29.0 mm to (82.0, 68.7), turned to 270 degrees
- moved D4 25.0 mm to (67.1, 71.3), turned to 0 degrees
- moved R9 20.5 mm to (69.4, 72.1), turned to 270 degrees
- moved U1 18.6 mm to (65.6, 104.1), turned to 180 degrees
- moved U3 17.1 mm to (77.8, 80.1)
- moved R4 17.1 mm to (69.0, 99.0), turned to 90 degrees
- moved D1 16.9 mm to (66.8, 99.5)
- moved C3 16.8 mm to (80.2, 80.2), turned to 90 degrees
- moved R7 16.1 mm to (55.8, 80.8)
- moved U4 11.3 mm to (74.0, 98.4), turned to 90 degrees
- moved R6 11.0 mm to (55.8, 83.3)
- moved J5 10.8 mm to (52.0, 99.5), turned to 180 degrees
- moved C2 9.74 mm to (70.8, 105.4), turned to 270 degrees
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Connections:
- J4 pad 6: SWD_DIO -> SWD_SWO
Routing:
- net GND: track 0.00 -> 119.6 mm, vias 0 -> 36
- net +3V3: track 0.00 -> 43.7 mm, vias 0 -> 21
- net +5V: track 0.00 -> 42.7 mm, vias 0 -> 4
- net FLASH_!HOLD: track 0.00 -> 30.8 mm, vias 0 -> 2
- net SPI2_SCK: track 0.00 -> 30.0 mm, vias 0 -> 3
- net SPI2_MISO: track 0.00 -> 29.1 mm, vias 0 -> 2
- net FLASH_!WP: track 0.00 -> 28.7 mm, vias 0 -> 2
- net USB_D+: track 0.00 -> 27.0 mm
- net NRST: track 0.00 -> 27.0 mm, vias 0 -> 2
- net SPI2_MOSI: track 0.00 -> 26.3 mm, vias 0 -> 2
- net USB_D-: track 0.00 -> 26.3 mm
- net ADC1_IN2: track 0.00 -> 25.7 mm, vias 0 -> 2
- net ADC1_IN1: track 0.00 -> 22.6 mm, vias 0 -> 2
- net SPI2_!CS: track 0.00 -> 21.6 mm, vias 0 -> 2
- net SWD_DIO: track 0.00 -> 21.6 mm
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- added copper zone on In2.Cu, net +3V3
- added copper zone on In1.Cu, net GND
Other:
- outline, holes or cut-outs redrawn
- copper layers 2 -> 4
- board text added: "+"
- board text added: "+3V3"
- board text added: "+5V"
- board text added: "3V3"
- board text added: "ACC"
- board text added: "ADC"
- board text added: "BOOT"
- board text added: "FLASH"
- board text added: "GND"
- board text added: "JLCJLCJLCJLC"
- board text added: "PWR"
- board text added: "SOIC8"
- board text added: "SWD"
- board text added: "TEMP"
- board text added: "TIM"
- board text added: "USB"
- board text added: "USR"
- board text added: "WAHLY Sensor Board J. Wahl"
- board text added: "v0.1"
